File: Carte/shieldBeagleBone.sch (KiCad schematic (older format))
At the start: 16 parts

Commit message: Added PushButton and PWM handlers (to be continued)
Parts:
- added C? (x2): C, symbol C
- added P?: Battery, symbol CONN_01X03
- added P?: LED_R_BACK, symbol CONN_01X02
- added P?: SONAR, symbol CONN_01X02
- added P?: ENCODER_R, symbol CONN_01X04
- added P?: ENCODER_L, symbol CONN_01X02
- added R?: R, symbol R
- added SW?: SW_PUSH, symbol SW_PUSH
- added SW?: SWITCH_INV, symbol SWITCH_INV
Connections:
- net Cmd_LED_STATUS: now also U?.11 (5A)
- net GND: now also C?.2, P?.1 (P1), P?.1 (P1), SW?.1, SW?.3
- net inputPower: now also C?.2, SW?.2
- net pushButton_RESET: now reaches U?.927 (GPIO_115)
- net pushButton_RESET: now also C?.1, SW?.2
- net TRIGGER: now reaches U?.928 (GPIO_123)
- net TRIGGER: now also P?.1 (P1)
- net ECHO: now reaches U?.929 (GPIO_121)
- net ECHO: now also P?.2 (P2)
- net at U?.10 (5Y): now also R?.2
- net at U?.12 (6Y): now also R?.2; no longer R?.2
- new net: C?.1, P?.2 (P2), SW?.1
- new net: P?.2 (P2), R?.1
- no-connect marks 6 -> 5
Other:
- moved on the sheet: P?, R?, U?
Changed lines of the file:
@@
 L RXEF050 U?
 U 1 1 57F50A69
-P 9050 700
-F 0 "U?" H 9650 550 60  0000 C CNN
-F 1 "RUEF135" H 9600 700 60  0000 C CNN
-F 2 "BeagleBone_FP:RXEF050" H 9050 700 60  0001 C CNN
-F 3 "" H 9050 700 60  0000 C CNN
-	1    9050 700
+P 7250 850
+F 0 "U?" H 7850 700 60  0000 C CNN
+F 1 "RUEF135" H 7800 850 60  0000 C CNN
+F 2 "BeagleBone_FP:RXEF050" H 7250 850 60  0001 C CNN
+F 3 "" H 7250 850 60  0000 C CNN
+	1    7250 850
 	1    0    0    -1
 $EndComp
@@
 	1    0    0    -1
 $EndComp
-Wire Wire Line
-	11050 650  11050 750
-Text GLabel 9050 850  0    39   Input ~ 0
+Text GLabel 7250 1000 0    39   Input ~ 0
 5V
 Text GLabel 2800 2400 2    39   Input ~ 0
@@
 Text GLabel 9100 2400 0    39   Input ~ 0
 5V
-Wire Wire Line
-	4500 1050 4500 1150
-Wire Wire Line
-	3950 1050 4500 1050
-Wire Wire Line
-	3950 1500 5600 1500
-Wire Wire Line
-	5600 1500 5600 1250
-Wire Wire Line
-	1000 1050 2750 1050
 Text GLabel 2750 1650 0    39   Input ~ 0
 DIRECTION_MOTOR_R
-Wire Wire Line
-	2100 1400 2350 1400
-Wire Wire Line
-	2350 1400 2350 1500
-Wire Wire Line
-	2350 1500 2750 1500
-Wire Wire Line
-	1000 1050 1000 1300
 Text GLabel 9100 3500 0    39   Input ~ 0
 motorEnable_L
@@
 	-1   0    0    1
 $EndComp
-Wire Wire Line
-	1000 2500 1150 2500
-Wire Wire Line
-	1150 2500 1150 2150
-Wire Wire Line
-	1150 2150 1000 2150
 Text GLabel 1150 2150 2    39   Input ~ 0
 GND
@@
 Text GLabel 1700 2400 0    39   Input ~ 0
 Cmd_LED_R
-Wire Wire Line
-	1000 2600 1400 2600
-Wire Wire Line
-	1400 2600 1400 2550
-Wire Wire Line
-	1000 2250 1000 2550
-Wire Wire Line
-	1000 2550 1400 2550
 Text GLabel 1700 2700 0    39   Input ~ 0
 Cmd_LED_L
@@
 	-1   0    0    1
 $EndComp
-Wire Wire Line
-	1000 3250 1150 3250
-Wire Wire Line
-	1150 3250 1150 2900
-Wire Wire Line
-	1150 2900 1000 2900
 Text GLabel 1150 2900 2    39   Input ~ 0
 GND
-Wire Wire Line
-	1000 3000 1400 3000
-Wire Wire Line
-	1400 2850 1400 3350
-Wire Wire Line
-	1400 3350 1000 3350
-Connection ~ 1400 3000
 NoConn ~ 1700 3000
 NoConn ~ 1700 3150
@@
 L R R?
 U 1 1 57F55147
-P 2950 2700
-F 0 "R?" V 3030 2700 50  0000 C CNN
-F 1 "R" V 2950 2700 50  0000 C CNN
-F 2 "" V 2880 2700 50  0000 C CNN
-F 3 "" H 2950 2700 50  0000 C CNN
-	1    2950 2700
+P 3600 3000
+F 0 "R?" V 3680 3000 50  0000 C CNN
+F 1 "R" V 3600 3000 50  0000 C CNN
+F 2 "" V 3530 3000 50  0000 C CNN
+F 3 "" H 3600 3000 50  0000 C CNN
+	1    3600 3000
 	0    1    1    0
 $EndComp
@@
 L CONN_01X02 P?
 U 1 1 57F551B8
-P 3300 2750
-F 0 "P?" H 3300 2900 50  0000 C CNN
-F 1 "LED_R_BACK" V 3400 2750 50  0000 C CNN
-F 2 "" H 3300 2750 50  0000 C CNN
-F 3 "" H 3300 2750 50  0000 C CNN
-	1    3300 2750
-	1    0    0    -1
-$EndComp
-Text GLabel 3100 2800 3    39   Input ~ 0
-GND
-NoConn ~ 2800 2850
-NoConn ~ 2800 3000
+P 3950 3050
+F 0 "P?" H 3950 3200 50  0000 C CNN
+F 1 "LED_R_BACK" V 4050 3050 50  0000 C CNN
+F 2 "" H 3950 3050 50  0000 C CNN
+F 3 "" H 3950 3050 50  0000 C CNN
+	1    3950 3050
+	1    0    0    -1
+$EndComp
+Text GLabel 3750 3100 3    39   Input ~ 0
+GND
 NoConn ~ 2800 3150
 NoConn ~ 2800 3300
-Text GLabel 10150 850  2    39   Input ~ 0
+Text GLabel 8350 1000 2    39   Input ~ 0
 inputPower
 Text GLabel 9100 4400 0    39   Input ~ 0
 Cmd_LED_STATUS
+Text GLabel 1550 4100 0    39   Input ~ 0
+GND
+Text GLabel 9100 4500 0    39   Input ~ 0
+pushButton_RESET
+Text GLabel 2550 4100 2    39   Input ~ 0
+pushButton_RESET
+Text Label 2300 3950 0    60   ~ 0
+Use_internal_pull-ups
+$Comp
+L SW_PUSH SW?
+U 1 1 57F78A18
+P 2050 4100
+F 0 "SW?" H 2200 4210 50  0000 C CNN
+F 1 "SW_PUSH" H 2050 4020 50  0000 C CNN
+F 2 "" H 2050 4100 50  0000 C CNN
+F 3 "" H 2050 4100 50  0000 C CNN
+	1    2050 4100
+	1    0    0    -1
+$EndComp
+$Comp
+L CONN_01X03 P?
+U 1 1 57F78BFD
+P 10450 750
+F 0 "P?" H 10450 900 50  0000 C CNN
+F 1 "Battery" V 10550 750 50  0000 C CNN
+F 2 "" H 10450 750 50  0000 C CNN
+F 3 "" H 10450 750 50  0000 C CNN
+	1    10450 750
+	1    0    0    -1
+$EndComp
+Text GLabel 10250 650  0    39   Input ~ 0
+GND
+$Comp
+L C C?
+U 1 1 57F78D95
+P 2050 4350
+F 0 "C?" H 2075 4450 50  0000 L CNN
+F 1 "C" H 2075 4250 50  0000 L CNN
+F 2 "" H 2088 4200 50  0000 C CNN
+F 3 "" H 2050 4350 50  0000 C CNN
+	1    2050 4350
+	0    1    1    0
+$EndComp
+$Comp
+L SWITCH_INV SW?
+U 1 1 57F78F93
+P 9750 850
+F 0 "SW?" H 9550 1000 50  0000 C CNN
+F 1 "SWITCH_INV" H 9600 700 50  0000 C CNN
+F 2 "" H 9750 850 50  0000 C CNN
+F 3 "" H 9750 850 50  0000 C CNN
+	1    9750 850
+	1    0    0    -1
+$EndComp
+Text GLabel 10250 950  2    39   Input ~ 0
+GND
+Text GLabel 9250 850  0    39   Input ~ 0
+inputPower
+$Comp
+L C C?
+U 1 1 57F79193
+P 9700 600
+F 0 "C?" H 9725 700 50  0000 L CNN
+F 1 "C" H 9725 500 50  0000 L CNN
+F 2 "" H 9738 450 50  0000 C CNN
+F 3 "" H 9700 600 50  0000 C CNN
+	1    9700 600
+	0    1    1    0
+$EndComp
+Text GLabel 2800 2850 2    39   Input ~ 0
+Cmd_LED_STATUS
+$Comp
+L R R?
+U 1 1 57F79824
+P 3600 2700
+F 0 "R?" V 3680 2700 50  0000 C CNN
+F 1 "R" V 3600 2700 50  0000 C CNN
+F 2 "" V 3530 2700 50  0000 C CNN
+F 3 "" H 3600 2700 50  0000 C CNN
+	1    3600 2700
+	0    1    1    0
+$EndComp
+$Comp
+L CONN_01X02 P?
+U 1 1 57F79880
+P 4100 2600
+F 0 "P?" H 4100 2750 50  0000 C CNN
+F 1 "LED_R_BACK" V 4200 2600 50  0000 C CNN
+F 2 "" H 4100 2600 50  0000 C CNN
+F 3 "" H 4100 2600 50  0000 C CNN
+	1    4100 2600
+	1    0    0    -1
+$EndComp
+Text GLabel 3900 2550 1    39   Input ~ 0
+GND
+Wire Wire Line
+	2800 2700 3450 2700
+Wire Wire Line
+	2800 3000 3450 3000
+Wire Wire Line
+	10050 750  10250 750
+Wire Wire Line
+	10050 600  10050 750
+Wire Wire Line
+	9850 600  10050 600
+Wire Wire Line
+	9250 600  9250 850
+Wire Wire Line
+	9550 600  9250 600
+Wire Wire Line
+	2350 4350 2350 4100
+Wire Wire Line
+	2200 4350 2350 4350
+Wire Wire Line
+	1750 4350 1750 4100
+Wire Wire Line
+	1900 4350 1750 4350
+Wire Wire Line
+	2350 4100 2550 4100
+Wire Wire Line
+	1750 4100 1550 4100
+Connection ~ 1400 3000
+Wire Wire Line
+	1400 3350 1000 3350
+Wire Wire Line
+	1400 2850 1400 3350
+Wire Wire Line
+	1000 3000 1400 3000
+Wire Wire Line
+	1150 2900 1000 2900
+Wire Wire Line
+	1150 3250 1150 2900
+Wire Wire Line
+	1000 3250 1150 3250
+Wire Wire Line
+	1000 2550 1400 2550
+Wire Wire Line
+	1000 2250 1000 2550
+Wire Wire Line
+	1400 2550 1400 2600
+Wire Wire Line
+	1400 2600 1000 2600
+Wire Wire Line
+	1150 2150 1000 2150
+Wire Wire Line
+	1150 2500 1150 2150
+Wire Wire Line
+	1000 2500 1150 2500
+Wire Wire Line
+	1000 1050 1000 1300
+Wire Wire Line
+	2350 1500 2750 1500
+Wire Wire Line
+	2350 1400 2350 1500
+Wire Wire Line
+	2100 1400 2350 1400
+Wire Wire Line
+	1000 1050 2750 1050
+Wire Wire Line
+	5600 1500 5600 1250
+Wire Wire Line
+	3950 1500 5600 1500
+Wire Wire Line
+	3950 1050 4500 1050
+Wire Wire Line
+	4500 1050 4500 1150
+Wire Wire Line
+	11050 650  11050 750
+Wire Wire Line
+	3750 2700 3900 2700
+Wire Wire Line
+	3900 2700 3900 2650
+NoConn ~ 10250 850
+$Comp
+L CONN_01X04 P?
+U 1 1 57F7B118
+P 1100 4900
+F 0 "P?" H 1100 5050 50  0000 C CNN
+F 1 "ENCODER_R" V 1200 4900 50  0000 C CNN
+F 2 "" H 1100 4900 50  0000 C CNN
+F 3 "" H 1100 4900 50  0000 C CNN
+	1    1100 4900
+	-1   0    0    -1
+$EndComp
+$Comp
+L CONN_01X02 P?
+U 1 1 57F7B215
+P 1100 5500
+F 0 "P?" H 1100 5650 50  0000 C CNN
+F 1 "ENCODER_L" V 1200 5500 50  0000 C CNN
+F 2 "" H 1100 5500 50  0000 C CNN
+F 3 "" H 1100 5500 50  0000 C CNN
+	1    1100 5500
+	-1   0    0    -1
+$EndComp
+$Comp
+L CONN_01X02 P?
+U 1 1 57F7A88E
+P 1150 6050
+F 0 "P?" H 1150 6200 50  0000 C CNN
+F 1 "SONAR" V 1250 6050 50  0000 C CNN
+F 2 "" H 1150 6050 50  0000 C CNN
+F 3 "" H 1150 6050 50  0000 C CNN
+	1    1150 6050
+	-1   0    0    -1
+$EndComp
+Text GLabel 1350 6000 2    39   Input ~ 0
+TRIGGER
+Text GLabel 1350 6100 2    39   Input ~ 0
+ECHO
+Text GLabel 9100 4600 0    39   Input ~ 0
+TRIGGER
+Text GLabel 9100 4700 0    39   Input ~ 0
+ECHO
 $EndSCHEMATC
